File: KICAD/PIC32MX_USBMSC_Driver.sch (KiCad schematic (older format))
At the start: 16 parts

Commit message: the circuit schematic up date
Parts:
- 10uF1: renamed from 10uF; value CP -> C?
- C3, C4, C5: renamed from 0.1uF; value C -> 0.1uF
- R1: renamed from 10K; value R -> 10K
- R2: renamed from R?; value R -> 330
- gave numbers to parts that had none: 10
Connections:
- no-connect marks 0 -> 12

Commit message: the circuit schematic update
Parts:
- C1: value C -> 0.1uF
- C2: value CP -> 10uF
- C6: renamed from 10uF1; value C? -> 10uF
Changed lines of the file:
@@
 EESchema Schematic File Version 4
+LIBS:PIC32MX_USBMSC_Driver-cache
 EELAYER 30 0
 EELAYER END
@@
 P 1600 6350
 F 0 "C1" H 1715 6391 43  0000 L CNN
-F 1 "C" H 1715 6310 43  0000 L CNN
+F 1 "0.1uF" H 1715 6310 43  0000 L CNN
 F 2 "" H 1638 6200 30  0000 C CNN
 F 3 "" H 1600 6350 60  0000 C CNN
@@
 P 2850 6350
 F 0 "C2" H 2968 6396 50  0000 L CNN
-F 1 "CP" H 2968 6305 50  0000 L CNN
+F 1 "10uF" H 2968 6305 50  0000 L CNN
 F 2 "" H 2888 6200 50  0000 C CNN
 F 3 "" H 2850 6350 50  0000 C CNN
@@
 $EndComp
 $Comp
-L mylib20161223:CP 10uF1
+L mylib20161223:CP C6
 U 1 1 5E2F104C
 P 7850 4000
-F 0 "10uF1" V 8000 4000 50  0000 C CNN
-F 1 "C?" V 7686 4000 50  0000 C CNN
+F 0 "C6" V 8000 4000 50  0000 C CNN
+F 1 "10uF" V 7686 4000 50  0000 C CNN
 F 2 "" H 7888 3850 50  0000 C CNN
 F 3 "" H 7850 4000 50  0000 C CNN

Commit message: the circuit schematic update
Parts:
- Y1: value Resonator_Small -> 4Mhz
Changed lines of the file:
@@
 P 2800 3800
 F 0 "Y1" V 2495 3750 50  0000 C CNN
-F 1 "Resonator_Small" V 2586 3750 50  0000 C CNN
+F 1 "4Mhz" V 2586 3750 50  0000 C CNN
 F 2 "" H 2775 3800 50  0001 C CNN
 F 3 "~" H 2775 3800 50  0001 C CNN

Commit message: amend debug prints around vUSBMSC & vSCSI
Parts:
- added C7: 10uF, symbol mylib20161223:CP
- added C8: 0.1uF, symbol mylib20161223:C
Connections:
- net +5.0V: now also C7.1, C8.2
- net GND: now also C7.2, C8.1
Changed lines of the file:
@@
 EESchema Schematic File Version 4
-LIBS:PIC32MX_USBMSC_Driver-cache
 EELAYER 30 0
 EELAYER END
@@
 L mylib20161223:+5.0V #PWR021
 U 1 1 5E318C4C
-P 8700 3600
-F 0 "#PWR021" H 8700 3525 30  0001 C CNN
-F 1 "+5.0V" H 8700 3738 30  0000 C CNN
-F 2 "" H 8700 3600 60  0000 C CNN
-F 3 "" H 8700 3600 60  0000 C CNN
-	1    8700 3600
+P 8700 3100
+F 0 "#PWR021" H 8700 3025 30  0001 C CNN
+F 1 "+5.0V" H 8700 3238 30  0000 C CNN
+F 2 "" H 8700 3100 60  0000 C CNN
+F 3 "" H 8700 3100 60  0000 C CNN
+	1    8700 3100
 	1    0    0    -1
 $EndComp
@@
 NoConn ~ 4300 4100
 NoConn ~ 7500 4500
+$Comp
+L mylib20161223:CP C7
+U 1 1 5E38BC5C
+P 8950 3250
+F 0 "C7" V 9200 3250 50  0000 C CNN
+F 1 "10uF" V 9100 3250 50  0000 C CNN
+F 2 "" H 8988 3100 50  0000 C CNN
+F 3 "" H 8950 3250 50  0000 C CNN
+	1    8950 3250
+	1    0    0    -1
+$EndComp
+$Comp
+L mylib20161223:C C8
+U 1 1 5E38CCA4
+P 9400 3250
+F 0 "C8" V 9163 3250 43  0000 C CNN
+F 1 "0.1uF" V 9244 3250 43  0000 C CNN
+F 2 "" H 9438 3100 30  0000 C CNN
+F 3 "" H 9400 3250 60  0000 C CNN
+	1    9400 3250
+	-1   0    0    1
+$EndComp
+Wire Wire Line
+	8700 3100 8950 3100
+Wire Wire Line
+	8950 3100 9400 3100
+Connection ~ 8950 3100
+Wire Wire Line
+	8700 3100 8700 3600
+Connection ~ 8700 3100
+$Comp
+L mylib20161223:GND #PWR024
+U 1 1 5E3919D8
+P 8950 3400
+F 0 "#PWR024" H 8950 3400 30  0001 C CNN
+F 1 "GND" H 8950 3330 30  0001 C CNN
+F 2 "" H 8950 3400 60  0000 C CNN
+F 3 "" H 8950 3400 60  0000 C CNN
+	1    8950 3400
+	1    0    0    -1
+$EndComp
+$Comp
+L mylib20161223:GND #PWR025
+U 1 1 5E391E01
+P 9400 3400
+F 0 "#PWR025" H 9400 3400 30  0001 C CNN
+F 1 "GND" H 9400 3330 30  0001 C CNN
+F 2 "" H 9400 3400 60  0000 C CNN
+F 3 "" H 9400 3400 60  0000 C CNN
+	1    9400 3400
+	1    0    0    -1
+$EndComp
 $EndSCHEMATC
